File: eagle/mlx90621_panel_shield.brd (EAGLE design)
At the start: 53.3 x 59.7 mm, 16 parts, among them J1 ARDUINO_R3_SHIELD

Commit message: Finalizado diseño de panel shield
Parts:
- removed U$6, U$7: MOUSE-BITES-4, mouse-bites:MOUSE-BITES-4
- added C3, C4, C5, C6: 100n, adafruit:C0603
- added JP2, JP3: (no value), SparkFun-Connectors:1X04
- added R3, R4, R5, R6: 10k, adafruit:R0603
- added S3, S4, S5, S6: STANDOFF_ELECTRICAL, SparkFun-Electromechanical:STANDOFF-ELECTRICAL
- added U$10, U$11, U$12, U$16, U$17, U$18: MOUSE-BITES-4, mouse-bites:MOUSE-BITES-4
- added U$14, U$8: MLX90621BAD, melexis:MLX90621
- added U$15, U$9: ZXCL260, melexis:VREG_SOT23-5
Connections:
- new net GND1: C3.2, C4.2, JP2.1, S3.P1, S4.P1, U$11.3, U$11.4, U$8.VSS, U$9.2
- new net GND2: C5.2, C6.2, JP3.1, S5.P1, S6.P1, U$14.VSS, U$15.2, U$17.3, U$17.4
- new net SCL1: JP2.4, R3.1, U$10.1, U$8.SCL
- new net SCL2: JP3.4, R5.1, U$14.SCL, U$16.1
- new net SDA1: JP2.3, R4.1, U$10.4, U$8.SDA
- new net SDA2: JP3.3, R6.1, U$14.SDA, U$16.4
- new net VCC1: C3.1, JP2.2, R3.2, R4.2, U$11.1, U$11.2, U$9.1, U$9.3
- new net VCC2: C5.1, JP3.2, R5.2, R6.2, U$15.1, U$15.3, U$17.1, U$17.2
- new net VDD1: C4.1, U$8.VDD, U$9.5
- new net VDD2: C6.1, U$14.VDD, U$15.5
- net GND: no longer J1.GND@2
Routing:
- net SDA2: track 0.00 -> 17.8 mm
- net SDA1: track 0.00 -> 17.8 mm
- net VCC2: track 0.00 -> 17.4 mm, vias 0 -> 2
- net VCC1: track 0.00 -> 17.4 mm, vias 0 -> 2
- net SCL1: track 0.00 -> 13.5 mm, vias 0 -> 1
- net SCL2: track 0.00 -> 13.5 mm, vias 0 -> 1
- net VDD1: track 0.00 -> 11.8 mm
- net VDD2: track 0.00 -> 11.8 mm
- net GND1: track 0.00 -> 3.51 mm, vias 0 -> 1
- net GND2: track 0.00 -> 2.86 mm, vias 0 -> 1
- net GND: vias 3 -> 7
- added copper zone on layer 1, net GND1
- added copper zone on layer 16, net GND1
- added copper zone on layer 1, net GND2
- added copper zone on layer 16, net GND2
Other:
- outline, holes or cut-outs redrawn

Commit message: Añadidos logos a shield
Parts:
- added E$1: (no value), DA_logo:DA_LOGO_10MM
- added E$2, E$3, E$4: (no value), DA_logo:DA_LOGO_5MM
Routing:
- net GND2: vias 1 -> 3
- net GND1: vias 1 -> 3
- net GND: vias 7 -> 8
Other:
- outline, holes or cut-outs redrawn
- board text added: "MLX90621 TEST SHIELD"
Changed lines of the file:
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@@
 <setting verticaltext="up"/>
 </settings>
-<grid distance="0.05" unitdist="inch" unit="inch" style="lines" multiple="1" display="yes" altdistance="0.00625" altunitdist="inch" altunit="inch"/>
+<grid distance="0.05" unitdist="inch" unit="inch" style="lines" multiple="1" display="yes" altdistance="0.0125" altunitdist="inch" altunit="inch"/>
 <layers>
 <layer number="1" name="Top" color="4" fill="1" visible="yes" active="yes"/>
@@
 <wire x1="10.95375" y1="8.89" x2="10.95375" y2="0.635" width="0" layer="20"/>
 <wire x1="10.95375" y1="0.635" x2="10.31875" y2="0" width="0" layer="20"/>
-<wire x1="35.56" y1="49.53" x2="35.56" y2="58.42" width="0" layer="20"/>
+<wire x1="35.56" y1="50.165" x2="35.56" y2="58.42" width="0" layer="20"/>
 <wire x1="12.84394375" y1="50.5529375" x2="11.90625" y2="48.142315625" width="0" layer="20" curve="42.510453"/>
 <wire x1="11.90625" y1="48.142315625" x2="11.90625" y2="46.51375" width="0" layer="20"/>
@@
 <wire x1="10.95375" y1="25.55875" x2="10.95375" y2="13.49375" width="0" layer="20"/>
 <wire x1="10.95375" y1="13.49375" x2="11.90625" y2="13.49375" width="0" layer="20"/>
+<text x="45.085" y="4.7625" size="1.4224" layer="21" font="vector" ratio="15" align="center">MLX90621
+TEST SHIELD</text>
 </plain>
 <attributes>
@@
 <element name="U$17" library="mouse-bites" package="MOUSE-BITES-4" value="MOUSE-BITES-4" x="34.925" y="10.16" rot="R270"/>
 <element name="U$18" library="mouse-bites" package="MOUSE-BITES-4" value="MOUSE-BITES-4" x="11.43" y="13.0175" rot="R270"/>
+<element name="E$1" library="DA_logo" package="DA_LOGO_10MM" value="" x="40.64" y="8.89"/>
+<element name="E$2" library="DA_logo" package="DA_LOGO_5MM" value="" x="24.13" y="13.335" rot="MR270"/>
+<element name="E$3" library="DA_logo" package="DA_LOGO_5MM" value="" x="24.4475" y="29.845" rot="MR270"/>
+<element name="E$4" library="DA_logo" package="DA_LOGO_5MM" value="" x="24.13" y="46.355" rot="MR270"/>
 </elements>
 <signals>
@@
 <via x="39.37" y="38.1" extent="1-16" drill="0.508"/>
 <via x="39.37" y="33.02" extent="1-16" drill="0.508"/>
+<via x="28.575" y="41.5925" extent="1-16" drill="0.3048"/>
 </signal>
 <signal name="VCC">
@@
 <vertex x="18.25625" y="33.655"/>
 <vertex x="35.56" y="33.655"/>
-<vertex x="35.56" y="22.225"/>
 </polygon>
+<via x="28.8925" y="25.0825" extent="1-16" drill="0.3048"/>
+<via x="26.9875" y="23.1775" extent="1-16" drill="0.3048"/>
 </signal>
 <signal name="VCC1">
@@
 <vertex x="35.56" y="17.145"/>
 </polygon>
+<via x="28.575" y="8.5725" extent="1-16" drill="0.3048"/>
+<via x="26.9875" y="6.6675" extent="1-16" drill="0.3048"/>
 <wire x1="34.2773" y1="7.3152" x2="34.925" y2="7.3152" width="0" layer="19" extent="1-1"/>
 </signal>
@@
 </board>
 </drawing>
+<compatibility>
+<note version="6.3" minversion="6.2.2" severity="warning">
+Since Version 6.2.2 text objects can contain more than one line,
+which will not be processed correctly with this version.
+</note>
+</compatibility>
 </eagle>
